Commit message: save launch

File: ws_moveit/src/mecademic_description/urdf/meca_500_r3.urdf.xacro (robot description, xacro)
@@ -160,41 +160,3 @@
     <origin xyz="0 0 0" rpy="0 0 0"/>
   </joint>
-  <!-- === ros2_control (optional Fake HW) === -->
-  <xacro:if value="$(arg use_fake_hw)">
-    <ros2_control name="FakeSystem" type="system">
-      <hardware>
-        <plugin>mock_components/GenericSystem</plugin>
-      </hardware>
-      <joint name="meca_axis_1_joint">
-        <command_interface name="position"/>
-        <state_interface   name="position"/>
-        <state_interface   name="velocity"/>
-      </joint>
-      <joint name="meca_axis_2_joint">
-        <command_interface name="position"/>
-        <state_interface   name="position"/>
-        <state_interface   name="velocity"/>
-      </joint>
-      <joint name="meca_axis_3_joint">
-        <command_interface name="position"/>
-        <state_interface   name="position"/>
-        <state_interface   name="velocity"/>
-      </joint>
-      <joint name="meca_axis_4_joint">
-        <command_interface name="position"/>
-        <state_interface   name="position"/>
-        <state_interface   name="velocity"/>
-      </joint>
-      <joint name="meca_axis_5_joint">
-        <command_interface name="position"/>
-        <state_interface   name="position"/>
-        <state_interface   name="velocity"/>
-      </joint>
-      <joint name="meca_axis_6_joint">
-        <command_interface name="position"/>
-        <state_interface   name="position"/>
-        <state_interface   name="velocity"/>
-      </joint>
-    </ros2_control>
-  </xacro:if>
 </robot>

File: ws_moveit/src/mecademic_moveit_config/config/meca_500_r3.ros2_control.xacro (robot description, xacro)
@@ -1,54 +1,55 @@
 <?xml version="1.0"?>
 <robot xmlns:xacro="http://www.ros.org/wiki/xacro">
-    <xacro:macro name="meca_500_r3_ros2_control" params="name initial_positions_file">
-        <xacro:property name="initial_positions" value="${xacro.load_yaml(initial_positions_file)['initial_positions']}"/>
-        <ros2_control name="meca500_fake_system" type="system">
-            <hardware>
-                <!-- By default, set up controllers for simulation. This won't work on real hardware -->
-                <plugin>mock_components/GenericSystem</plugin>
-            </hardware>
-            <joint name="meca_axis_1_joint">
-                <command_interface name="position"/>
-                <state_interface name="position">
-                  <param name="initial_value">${initial_positions['meca_axis_1_joint']}</param>
-                </state_interface>
-                <state_interface name="velocity"/>
-            </joint>
-            <joint name="meca_axis_2_joint">
-                <command_interface name="position"/>
-                <state_interface name="position">
-                  <param name="initial_value">${initial_positions['meca_axis_2_joint']}</param>
-                </state_interface>
-                <state_interface name="velocity"/>
-            </joint>
-            <joint name="meca_axis_3_joint">
-                <command_interface name="position"/>
-                <state_interface name="position">
-                  <param name="initial_value">${initial_positions['meca_axis_3_joint']}</param>
-                </state_interface>
-                <state_interface name="velocity"/>
-            </joint>
-            <joint name="meca_axis_4_joint">
-                <command_interface name="position"/>
-                <state_interface name="position">
-                  <param name="initial_value">${initial_positions['meca_axis_4_joint']}</param>
-                </state_interface>
-                <state_interface name="velocity"/>
-            </joint>
-            <joint name="meca_axis_5_joint">
-                <command_interface name="position"/>
-                <state_interface name="position">
-                  <param name="initial_value">${initial_positions['meca_axis_5_joint']}</param>
-                </state_interface>
-                <state_interface name="velocity"/>
-            </joint>
-            <joint name="meca_axis_6_joint">
-                <command_interface name="position"/>
-                <state_interface name="position">
-                  <param name="initial_value">${initial_positions['meca_axis_6_joint']}</param>
-                </state_interface>
-                <state_interface name="velocity"/>
-            </joint>
-        </ros2_control>
-    </xacro:macro>
+  <!-- Macro für ros2_control-Setup -->
+  <xacro:macro name="meca_500_r3_ros2_control" params="name initial_positions_file">
+    <!-- YAML mit Startpositionen laden -->
+    <xacro:property name="initial_positions" value="${xacro.load_yaml(initial_positions_file)['initial_positions']}"/>
+    <ros2_control name="${name}" type="system">
+      <hardware>
+        <plugin>mock_components/GenericSystem</plugin>
+      </hardware>
+      <joint name="meca_axis_1_joint">
+        <command_interface name="position"/>
+        <state_interface name="position">
+          <param name="initial_value">${initial_positions['meca_axis_1_joint']}</param>
+        </state_interface>
+        <state_interface name="velocity"/>
+      </joint>
+      <joint name="meca_axis_2_joint">
+        <command_interface name="position"/>
+        <state_interface name="position">
+          <param name="initial_value">${initial_positions['meca_axis_2_joint']}</param>
+        </state_interface>
+        <state_interface name="velocity"/>
+      </joint>
+      <joint name="meca_axis_3_joint">
+        <command_interface name="position"/>
+        <state_interface name="position">
+          <param name="initial_value">${initial_positions['meca_axis_3_joint']}</param>
+        </state_interface>
+        <state_interface name="velocity"/>
+      </joint>
+      <joint name="meca_axis_4_joint">
+        <command_interface name="position"/>
+        <state_interface name="position">
+          <param name="initial_value">${initial_positions['meca_axis_4_joint']}</param>
+        </state_interface>
+        <state_interface name="velocity"/>
+      </joint>
+      <joint name="meca_axis_5_joint">
+        <command_interface name="position"/>
+        <state_interface name="position">
+          <param name="initial_value">${initial_positions['meca_axis_5_joint']}</param>
+        </state_interface>
+        <state_interface name="velocity"/>
+      </joint>
+      <joint name="meca_axis_6_joint">
+        <command_interface name="position"/>
+        <state_interface name="position">
+          <param name="initial_value">${initial_positions['meca_axis_6_joint']}</param>
+        </state_interface>
+        <state_interface name="velocity"/>
+      </joint>
+    </ros2_control>
+  </xacro:macro>
 </robot>

File: ws_moveit/src/mecademic_moveit_config/config/meca_500_r3.urdf.xacro (robot description, xacro)
@@ -1,9 +1,9 @@
 <?xml version="1.0"?>
 <robot xmlns:xacro="http://www.ros.org/wiki/xacro" name="meca_500_r3">
-    <xacro:arg name="initial_positions_file" default="initial_positions.yaml" />
-    <!-- Import meca_500_r3 urdf file -->
-    <xacro:include filename="$(find mecademic_description)/urdf/meca_500_r3.urdf.xacro" />
-    <!-- Import control_xacro -->
-    <xacro:include filename="meca_500_r3.ros2_control.xacro" />
-    <xacro:meca_500_r3_ros2_control name="FakeSystem" initial_positions_file="$(arg initial_positions_file)"/>
+  <xacro:arg name="initial_positions_file" default="$(find mecademic_moveit_config)/config/initial_positions.yaml" />
+  <!-- Include core geometry and visual URDF -->
+  <xacro:include filename="$(find mecademic_description)/urdf/meca_500_r3.urdf.xacro"/>
+  <!-- ros2_control (FakeSystem / real system later) -->
+  <xacro:include filename="$(find mecademic_moveit_config)/config/meca_500_r3.ros2_control.xacro"/>
+  <xacro:meca_500_r3_ros2_control name="FakeSystem" initial_positions_file="$(arg initial_positions_file)"/>
 </robot>
