Commit message: update files

File: ws_moveit/src/mecademic_moveit_config/config/meca_500_r3.ros2_control.xacro (robot description, xacro)
@@ -1,43 +1,54 @@
 <?xml version="1.0"?>
 <robot xmlns:xacro="http://www.ros.org/wiki/xacro">
-  <xacro:macro name="meca_500_r3_ros2_control" params="name">
-    <ros2_control name="${name}" type="system">
-      <hardware>
-        <!-- ✅ Fake ROS2 Control – wie früher, stabil für Simulation -->
-        <plugin>ros2_control_demo_hardware/GenericSystem</plugin>
-        <param name="fake_sensor_commands">true</param>
-      </hardware>
-      <!-- ✅ Keine initial_positions nötig, Fake hat Defaults -->
-      <joint name="meca_axis_1_joint">
-        <command_interface name="position" />
-        <state_interface name="position" />
-        <state_interface name="velocity" />
-      </joint>
-      <joint name="meca_axis_2_joint">
-        <command_interface name="position" />
-        <state_interface name="position" />
-        <state_interface name="velocity" />
-      </joint>
-      <joint name="meca_axis_3_joint">
-        <command_interface name="position" />
-        <state_interface name="position" />
-        <state_interface name="velocity" />
-      </joint>
-      <joint name="meca_axis_4_joint">
-        <command_interface name="position" />
-        <state_interface name="position" />
-        <state_interface name="velocity" />
-      </joint>
-      <joint name="meca_axis_5_joint">
-        <command_interface name="position" />
-        <state_interface name="position" />
-        <state_interface name="velocity" />
-      </joint>
-      <joint name="meca_axis_6_joint">
-        <command_interface name="position" />
-        <state_interface name="position" />
-        <state_interface name="velocity" />
-      </joint>
-    </ros2_control>
-  </xacro:macro>
+    <xacro:macro name="meca_500_r3_ros2_control" params="name initial_positions_file">
+        <xacro:property name="initial_positions" value="${xacro.load_yaml(initial_positions_file)['initial_positions']}"/>
+        <ros2_control name="meca500_fake_system" type="system">
+            <hardware>
+                <!-- By default, set up controllers for simulation. This won't work on real hardware -->
+                <plugin>mock_components/GenericSystem</plugin>
+            </hardware>
+            <joint name="meca_axis_1_joint">
+                <command_interface name="position"/>
+                <state_interface name="position">
+                  <param name="initial_value">${initial_positions['meca_axis_1_joint']}</param>
+                </state_interface>
+                <state_interface name="velocity"/>
+            </joint>
+            <joint name="meca_axis_2_joint">
+                <command_interface name="position"/>
+                <state_interface name="position">
+                  <param name="initial_value">${initial_positions['meca_axis_2_joint']}</param>
+                </state_interface>
+                <state_interface name="velocity"/>
+            </joint>
+            <joint name="meca_axis_3_joint">
+                <command_interface name="position"/>
+                <state_interface name="position">
+                  <param name="initial_value">${initial_positions['meca_axis_3_joint']}</param>
+                </state_interface>
+                <state_interface name="velocity"/>
+            </joint>
+            <joint name="meca_axis_4_joint">
+                <command_interface name="position"/>
+                <state_interface name="position">
+                  <param name="initial_value">${initial_positions['meca_axis_4_joint']}</param>
+                </state_interface>
+                <state_interface name="velocity"/>
+            </joint>
+            <joint name="meca_axis_5_joint">
+                <command_interface name="position"/>
+                <state_interface name="position">
+                  <param name="initial_value">${initial_positions['meca_axis_5_joint']}</param>
+                </state_interface>
+                <state_interface name="velocity"/>
+            </joint>
+            <joint name="meca_axis_6_joint">
+                <command_interface name="position"/>
+                <state_interface name="position">
+                  <param name="initial_value">${initial_positions['meca_axis_6_joint']}</param>
+                </state_interface>
+                <state_interface name="velocity"/>
+            </joint>
+        </ros2_control>
+    </xacro:macro>
 </robot>

File: ws_moveit/src/mecademic_moveit_config/config/meca_500_r3.urdf.xacro (robot description, xacro)
@@ -1,207 +1,9 @@
 <?xml version="1.0"?>
-<robot name="meca_500_r3" xmlns:xacro="http://www.ros.org/wiki/xacro">
-  <xacro:arg name="use_fake_hw" default="true"/>
-  <!-- Dummy Root -->
-  <link name="meca_mount"/>
-  <joint name="meca_mount_to_base" type="fixed">
-    <parent link="meca_mount"/>
-    <child  link="meca_base_link"/>
-    <origin xyz="0 0 0" rpy="0 0 0"/>
-  </joint>
-  <!-- === Base link === -->
-  <link name="meca_base_link">
-    <visual>
-      <geometry>
-        <mesh filename="package://mecademic_description/meshes/meca_500_r3_base.dae"/>
-      </geometry>
-    </visual>
-    <collision>
-      <geometry>
-        <mesh filename="package://mecademic_description/meshes/meca_500_r3_base_collision.stl"/>
-      </geometry>
-    </collision>
-    <inertial>
-      <origin xyz="0 0 0" rpy="0 0 0"/>
-      <mass value="1.0"/>
-      <inertia ixx="0.001" ixy="0" ixz="0" iyy="0.001" iyz="0" izz="0.001"/>
-    </inertial>
-  </link>
-  <!-- === Joint 1 === -->
-  <link name="meca_axis_1_link">
-    <visual>
-      <geometry><mesh filename="package://mecademic_description/meshes/meca_500_r3_j1.dae"/></geometry>
-    </visual>
-    <collision>
-      <geometry><mesh filename="package://mecademic_description/meshes/meca_500_r3_j1_collision.stl"/></geometry>
-    </collision>
-    <inertial>
-      <origin xyz="0 0 0" rpy="0 0 0"/>
-      <mass value="0.5"/>
-      <inertia ixx="0.0005" ixy="0" ixz="0" iyy="0.0005" iyz="0" izz="0.0005"/>
-    </inertial>
-  </link>
-  <joint name="meca_axis_1_joint" type="revolute">
-    <parent link="meca_base_link"/>
-    <child  link="meca_axis_1_link"/>
-    <origin xyz="0.012498 0 0.091" rpy="0 0 0"/>
-    <axis xyz="0 0 1"/>
-    <limit effort="10.0" velocity="2.61799" lower="-3.05433" upper="3.05433"/>
-  </joint>
-  <!-- === Joint 2 === -->
-  <link name="meca_axis_2_link">
-    <visual>
-      <geometry><mesh filename="package://mecademic_description/meshes/meca_500_r3_j2.dae"/></geometry>
-    </visual>
-    <collision>
-      <geometry><mesh filename="package://mecademic_description/meshes/meca_500_r3_j2_collision.stl"/></geometry>
-    </collision>
-    <inertial>
-      <origin xyz="0 0 0" rpy="0 0 0"/>
-      <mass value="0.4"/>
-      <inertia ixx="0.0004" ixy="0" ixz="0" iyy="0.0004" iyz="0" izz="0.0004"/>
-    </inertial>
-  </link>
-  <joint name="meca_axis_2_joint" type="revolute">
-    <parent link="meca_axis_1_link"/>
-    <child  link="meca_axis_2_link"/>
-    <origin xyz="0 0 0.044" rpy="0 0 0"/>
-    <axis xyz="0 1 0"/>
-    <limit effort="10.0" velocity="2.61799" lower="-1.22173" upper="1.5708"/>
-  </joint>
-  <!-- === Joint 3 === -->
-  <link name="meca_axis_3_link">
-    <visual>
-      <geometry><mesh filename="package://mecademic_description/meshes/meca_500_r3_j3.dae"/></geometry>
-    </visual>
-    <collision>
-      <geometry><mesh filename="package://mecademic_description/meshes/meca_500_r3_j3_collision.stl"/></geometry>
-    </collision>
-    <inertial>
-      <origin xyz="0 0 0" rpy="0 0 0"/>
-      <mass value="0.3"/>
-      <inertia ixx="0.0003" ixy="0" ixz="0" iyy="0.0003" iyz="0" izz="0.0003"/>
-    </inertial>
-  </link>
-  <joint name="meca_axis_3_joint" type="revolute">
-    <parent link="meca_axis_2_link"/>
-    <child  link="meca_axis_3_link"/>
-    <origin xyz="0 0 0.135" rpy="0 0 0"/>
-    <axis xyz="0 1 0"/>
-    <limit effort="10.0" velocity="3.14159" lower="-2.35619" upper="1.22173"/>
-  </joint>
-  <!-- === Joint 4 === -->
-  <link name="meca_axis_4_link">
-    <visual>
-      <geometry><mesh filename="package://mecademic_description/meshes/meca_500_r3_j4.dae"/></geometry>
-    </visual>
-    <collision>
-      <geometry><mesh filename="package://mecademic_description/meshes/meca_500_r3_j4_collision.stl"/></geometry>
-    </collision>
-    <inertial>
-      <origin xyz="0 0 0" rpy="0 0 0"/>
-      <mass value="0.25"/>
-      <inertia ixx="0.00025" ixy="0" ixz="0" iyy="0.00025" iyz="0" izz="0.00025"/>
-    </inertial>
-  </link>
-  <joint name="meca_axis_4_joint" type="revolute">
-    <parent link="meca_axis_3_link"/>
-    <child  link="meca_axis_4_link"/>
-    <origin xyz="0 0 0.038" rpy="0 0 0"/>
-    <axis xyz="1 0 0"/>
-    <limit effort="10.0" velocity="5.23599" lower="-2.96706" upper="2.96706"/>
-  </joint>
-  <!-- === Joint 5 === -->
-  <link name="meca_axis_5_link">
-    <visual>
-      <geometry><mesh filename="package://mecademic_description/meshes/meca_500_r3_j5.dae"/></geometry>
-    </visual>
-    <collision>
-      <geometry><mesh filename="package://mecademic_description/meshes/meca_500_r3_j5_collision.stl"/></geometry>
-    </collision>
-    <inertial>
-      <origin xyz="0 0 0" rpy="0 0 0"/>
-      <mass value="0.2"/>
-      <inertia ixx="0.0002" ixy="0" ixz="0" iyy="0.0002" iyz="0" izz="0.0002"/>
-    </inertial>
-  </link>
-  <joint name="meca_axis_5_joint" type="revolute">
-    <parent link="meca_axis_4_link"/>
-    <child  link="meca_axis_5_link"/>
-    <origin xyz="0.12 0 0" rpy="0 0 0"/>
-    <axis xyz="0 1 0"/>
-    <limit effort="10.0" velocity="5.23599" lower="-2.00713" upper="2.00713"/>
-  </joint>
-  <!-- === Joint 6 === -->
-  <link name="meca_axis_6_link">
-    <visual>
-      <geometry><mesh filename="package://mecademic_description/meshes/meca_500_r3_j6.dae"/></geometry>
-    </visual>
-    <collision>
-      <geometry><mesh filename="package://mecademic_description/meshes/meca_500_r3_j6_collision.stl"/></geometry>
-    </collision>
-    <inertial>
-      <origin xyz="0 0 0" rpy="0 0 0"/>
-      <mass value="0.15"/>
-      <inertia ixx="0.00015" ixy="0" ixz="0.00015" iyy="0.00015" iyz="0" izz="0.00015"/>
-    </inertial>
-  </link>
-  <joint name="meca_axis_6_joint" type="revolute">
-    <parent link="meca_axis_5_link"/>
-    <child  link="meca_axis_6_link"/>
-    <origin xyz="0.07 0 0" rpy="0 0 0"/>
-    <axis xyz="1 0 0"/>
-    <limit effort="10.0" velocity="8.72665" lower="-3.14159" upper="3.14159"/>
-  </joint>
-  <!-- === Tool-Mount === -->
-  <link name="tool_mount"/>
-  <joint name="tool_mount_joint" type="fixed">
-    <parent link="meca_axis_6_link"/>
-    <child  link="tool_mount"/>
-    <origin xyz="0 0 0" rpy="0 0 0"/>
-  </joint>
-  <!-- === Neutral TCP === -->
-  <link name="tcp"/>
-  <joint name="tcp_joint" type="fixed">
-    <parent link="tool_mount"/>
-    <child  link="tcp"/>
-    <origin xyz="0 0 0" rpy="0 0 0"/>
-  </joint>
-  <!-- === ros2_control (optional Fake HW) === -->
-  <xacro:if value="$(arg use_fake_hw)">
-    <ros2_control name="FakeSystem" type="system">
-      <hardware>
-        <plugin>mock_components/GenericSystem</plugin>
-      </hardware>
-      <joint name="meca_axis_1_joint">
-        <command_interface name="position"/>
-        <state_interface   name="position"/>
-        <state_interface   name="velocity"/>
-      </joint>
-      <joint name="meca_axis_2_joint">
-        <command_interface name="position"/>
-        <state_interface   name="position"/>
-        <state_interface   name="velocity"/>
-      </joint>
-      <joint name="meca_axis_3_joint">
-        <command_interface name="position"/>
-        <state_interface   name="position"/>
-        <state_interface   name="velocity"/>
-      </joint>
-      <joint name="meca_axis_4_joint">
-        <command_interface name="position"/>
-        <state_interface   name="position"/>
-        <state_interface   name="velocity"/>
-      </joint>
-      <joint name="meca_axis_5_joint">
-        <command_interface name="position"/>
-        <state_interface   name="position"/>
-        <state_interface   name="velocity"/>
-      </joint>
-      <joint name="meca_axis_6_joint">
-        <command_interface name="position"/>
-        <state_interface   name="position"/>
-        <state_interface   name="velocity"/>
-      </joint>
-    </ros2_control>
-  </xacro:if>
+<robot xmlns:xacro="http://www.ros.org/wiki/xacro" name="meca_500_r3">
+    <xacro:arg name="initial_positions_file" default="initial_positions.yaml" />
+    <!-- Import meca_500_r3 urdf file -->
+    <xacro:include filename="$(find mecademic_description)/urdf/meca_500_r3.urdf.xacro" />
+    <!-- Import control_xacro -->
+    <xacro:include filename="meca_500_r3.ros2_control.xacro" />
+    <xacro:meca_500_r3_ros2_control name="FakeSystem" initial_positions_file="$(arg initial_positions_file)"/>
 </robot>
