Commit message: fix robot model

File: ws_moveit/src/omron_viper_description/urdf/omron_viper.urdf.xacro (robot description, xacro)
@@ -1,159 +1,147 @@
 <?xml version="1.0"?>
-<robot name="ADEPT_VIPER_S650">
-  <!-- ===== Welt-Mount ===== -->
+<robot name="omron_viper_s650">
+  <!-- Welt -->
   <link name="world_mount"/>
-  <joint name="world_mount_to_link1" type="fixed">
+  <joint name="world_to_base" type="fixed">
     <parent link="world_mount"/>
     <child  link="Adept_Viper_s650_Link1"/>
     <origin xyz="0 0 0" rpy="0 0 0"/>
   </joint>
-  <!-- ===== LINKS ===== -->
+  <!-- Materialien -->
+  <material name="White"><color rgba="1 1 1 1"/></material>
+  <material name="Blue"><color rgba="0 0 1 1"/></material>
+  <material name="Red"><color rgba="1 0 0 1"/></material>
+  <material name="Green"><color rgba="0 1 0 1"/></material>
+  <material name="Gray"><color rgba="0.4 0.4 0.4 1"/></material>
+  <!-- LINKS (alle rpy=0) -->
   <link name="Adept_Viper_s650_Link1">
-    <visual>
-      <origin xyz="0 0 0" rpy="0 0 0"/>
-      <geometry>
-        <mesh filename="package://omron_viper_description/meshes/visual/Adept_Viper_650_Link1.stl"/>
-      </geometry>
-    </visual>
-    <collision>
-      <origin xyz="0 0 0" rpy="0 0 0"/>
-      <geometry>
-        <mesh filename="package://omron_viper_description/meshes/collision/Adept_Viper_650_Link1.stl"/>
-      </geometry>
-    </collision>
+    <visual><origin xyz="0 0 0" rpy="0 0 0"/><geometry>
+      <mesh filename="package://omron_viper_description/meshes/visual/Adept_Viper_650_Link1.stl"/>
+    </geometry><material name="White"/></visual>
+    <collision><origin xyz="0 0 0" rpy="0 0 0"/><geometry>
+      <mesh filename="package://omron_viper_description/meshes/collision/Adept_Viper_650_Link1.stl"/>
+    </geometry><material name="Blue"/></collision>
   </link>
   <link name="Adept_Viper_s650_Link2">
-    <visual>
-      <origin xyz="0 0 0" rpy="0 1.5714 0"/>
-      <geometry>
-        <mesh filename="package://omron_viper_description/meshes/visual/Adept_Viper_650_Link2.stl"/>
-      </geometry>
-    </visual>
-    <collision>
-      <origin xyz="0 0 0" rpy="0 1.5714 0"/>
-      <geometry>
-        <mesh filename="package://omron_viper_description/meshes/collision/Adept_Viper_650_Link2.stl"/>
-      </geometry>
-    </collision>
+    <visual><origin xyz="0 0 0" rpy="0 0 0"/><geometry>
+      <mesh filename="package://omron_viper_description/meshes/visual/Adept_Viper_650_Link2.stl"/>
+    </geometry><material name="Red"/></visual>
+    <collision><origin xyz="0 0 0" rpy="0 0 0"/><geometry>
+      <mesh filename="package://omron_viper_description/meshes/collision/Adept_Viper_650_Link2.stl"/>
+    </geometry><material name="Green"/></collision>
   </link>
   <link name="Adept_Viper_s650_Link3">
     <visual>
-      <origin xyz="0 0 0" rpy="0 -1.5714 0"/>
+      <!-- Mesh 90° um Y drehen -->
+      <origin xyz="0 0 0" rpy="0 1.5708 0"/>
       <geometry>
         <mesh filename="package://omron_viper_description/meshes/visual/Adept_Viper_650_Link3.stl"/>
       </geometry>
+      <material name="White"/>
     </visual>
     <collision>
-      <origin xyz="0 0 0" rpy="0 -1.5714 0"/>
+      <origin xyz="0 0 0" rpy="0 1.5708 0"/>
       <geometry>
         <mesh filename="package://omron_viper_description/meshes/collision/Adept_Viper_650_Link3.stl"/>
       </geometry>
+      <material name="Blue"/>
     </collision>
   </link>
-  <link name="Adept_Viper_s650_Link4">
-    <visual>
-      <origin xyz="0 0 0" rpy="0 -1.5714 0"/>
-      <geometry>
-        <mesh filename="package://omron_viper_description/meshes/visual/Adept_Viper_650_Link4.stl"/>
-      </geometry>
-    </visual>
-    <collision>
-      <origin xyz="0 0 0" rpy="0 -1.5714 0"/>
-      <geometry>
-        <mesh filename="package://omron_viper_description/meshes/collision/Adept_Viper_650_Link4.stl"/>
-      </geometry>
-    </collision>
-  </link>
-  <link name="Adept_Viper_s650_Link5">
-    <visual>
-      <origin xyz="0 0 0" rpy="0 -1.5714 0"/>
-      <geometry>
-        <mesh filename="package://omron_viper_description/meshes/visual/Adept_Viper_650_Link5.stl"/>
-      </geometry>
-    </visual>
-    <collision>
-      <origin xyz="0 0 0" rpy="0 -1.5714 0"/>
-      <geometry>
-        <mesh filename="package://omron_viper_description/meshes/collision/Adept_Viper_650_Link5.stl"/>
-      </geometry>
-    </collision>
-  </link>
-  <link name="Adept_Viper_s650_Link6">
-    <visual>
-      <origin xyz="0 0 0" rpy="0 -1.5714 0"/>
-      <geometry>
-        <mesh filename="package://omron_viper_description/meshes/visual/Adept_Viper_650_Link6.stl"/>
-      </geometry>
-    </visual>
-    <collision>
-      <origin xyz="0 0 0" rpy="0 -1.5714 0"/>
-      <geometry>
-        <mesh filename="package://omron_viper_description/meshes/collision/Adept_Viper_650_Link6.stl"/>
-      </geometry>
-    </collision>
-  </link>
-  <link name="Adept_Viper_650_Interface_Plate">
-    <visual>
-      <origin xyz="0 0 0" rpy="0 -1.5714 0"/>
-      <geometry>
-        <mesh filename="package://omron_viper_description/meshes/visual/Adept_Viper_650_Interface_Plate.stl"/>
-      </geometry>
-    </visual>
-    <collision>
-      <origin xyz="0 0 0" rpy="0 -1.5714 0"/>
-      <geometry>
-        <mesh filename="package://omron_viper_description/meshes/collision/Adept_Viper_650_Interface_Plate.stl"/>
-      </geometry>
-    </collision>
-  </link>
-  <!-- ===== JOINTS (Maße aus Datasheet) ===== -->
+<!-- Link4 -->
+<link name="Adept_Viper_s650_Link4">
+  <visual>
+    <origin xyz="0 0 0" rpy="0 -1.5708 0"/>
+    <geometry><mesh filename="package://omron_viper_description/meshes/visual/Adept_Viper_650_Link4.stl"/></geometry>
+    <material name="Red"/>
+  </visual>
+  <collision>
+    <origin xyz="0 0 0" rpy="0 -1.5708 0"/>
+    <geometry><mesh filename="package://omron_viper_description/meshes/collision/Adept_Viper_650_Link4.stl"/></geometry>
+    <material name="Blue"/>
+  </collision>
+</link>
+<!-- Link5 -->
+<link name="Adept_Viper_s650_Link5">
+  <visual>
+    <origin xyz="0 0 0" rpy="0 -1.5708 0"/>
+    <geometry><mesh filename="package://omron_viper_description/meshes/visual/Adept_Viper_650_Link5.stl"/></geometry>
+    <material name="Blue"/>
+  </visual>
+  <collision>
+    <origin xyz="0 0 0" rpy="0 -1.5708 0"/>
+    <geometry><mesh filename="package://omron_viper_description/meshes/collision/Adept_Viper_650_Link5.stl"/></geometry>
+    <material name="Blue"/>
+  </collision>
+</link>
+<!-- Link6 -->
+<link name="Adept_Viper_s650_Link6">
+  <visual>
+    <origin xyz="0 0 0" rpy="0 -1.5708 0"/>
+    <geometry><mesh filename="package://omron_viper_description/meshes/visual/Adept_Viper_650_Link6.stl"/></geometry>
+    <material name="Blue"/>
+  </visual>
+  <collision>
+    <origin xyz="0 0 0" rpy="0 -1.5708 0"/>
+    <geometry><mesh filename="package://omron_viper_description/meshes/collision/Adept_Viper_650_Link6.stl"/></geometry>
+    <material name="Blue"/>
+  </collision>
+</link>
+<!-- Interface Plate -->
+<link name="Adept_Viper_650_Interface_Plate">
+  <visual>
+    <origin xyz="0 0 0" rpy="0 -1.5708 0"/>
+    <geometry><mesh filename="package://omron_viper_description/meshes/visual/Adept_Viper_650_Interface_Plate.stl"/></geometry>
+    <material name="Gray"/>
+  </visual>
+  <collision>
+    <origin xyz="0 0 0" rpy="0 -1.5708 0"/>
+    <geometry><mesh filename="package://omron_viper_description/meshes/collision/Adept_Viper_650_Interface_Plate.stl"/></geometry>
+    <material name="Gray"/>
+  </collision>
+</link>
+  <!-- JOINTS (rein nach Datenblatt) -->
   <joint name="joint_1" type="revolute">
-    <!-- Basis-Flansch -> J2 Achse: 203 mm -->
-    <origin xyz="0 0 0.203" rpy="0 0 0"/>
     <parent link="Adept_Viper_s650_Link1"/>
     <child  link="Adept_Viper_s650_Link2"/>
+    <origin xyz="0 0 0.203" rpy="0 0 0"/>
     <axis xyz="0 0 1"/>
-    <limit effort="100" velocity="5.72468" lower="-2.9670" upper="2.9670"/>
+    <limit effort="100" velocity="5.72468" lower="-2.96706" upper="2.96706"/>
   </joint>
   <joint name="joint_2" type="revolute">
-    <!-- lokaler Versatz am Link2-Bauteil -->
-    <origin xyz="0.074 0 0.18795" rpy="0 0 0"/>
     <parent link="Adept_Viper_s650_Link2"/>
     <child  link="Adept_Viper_s650_Link3"/>
+    <origin xyz="0.074 0 0.132" rpy="0 0 0"/>
     <axis xyz="0 1 0"/>
-    <limit effort="100" velocity="5.235" lower="-3.31613" upper="0.7854"/>
+    <limit effort="100" velocity="5.23599" lower="-3.31613" upper="0.78540"/>
   </joint>
   <joint name="joint_3" type="revolute">
-    <!-- J2 -> J3: 270 mm -->
-    <origin xyz="0.270 0 0" rpy="0 0 0"/>
     <parent link="Adept_Viper_s650_Link3"/>
     <child  link="Adept_Viper_s650_Link4"/>
+    <origin xyz="0.270 0 0" rpy="0 0 0"/>
     <axis xyz="0 1 0"/>
-    <limit effort="100" velocity="6.544" lower="-0.50615" upper="4.468053"/>
+    <limit effort="100" velocity="6.54498" lower="-0.50615" upper="4.46805"/>
   </joint>
   <joint name="joint_4" type="revolute">
-    <!-- J3 -> J4: 295 mm, lokal -0.090 in X -->
-    <origin xyz="-0.090 0 0.295" rpy="0 0 0"/>
     <parent link="Adept_Viper_s650_Link4"/>
     <child  link="Adept_Viper_s650_Link5"/>
+    <origin xyz="-0.090 0 0.295" rpy="0 0 0"/>
     <axis xyz="0 0 1"/>
-    <limit effort="100" velocity="6.544" lower="-3.31613" upper="3.316133"/>
+    <limit effort="100" velocity="6.54498" lower="-3.31613" upper="3.31613"/>
   </joint>
   <joint name="joint_5" type="revolute">
-    <origin xyz="0 0 0" rpy="0 0 0"/>
     <parent link="Adept_Viper_s650_Link5"/>
     <child  link="Adept_Viper_s650_Link6"/>
+    <origin xyz="0 0 0" rpy="0 0 0"/>
     <axis xyz="0 1 0"/>
-    <limit effort="100" velocity="6.544" lower="-2.0944" upper="2.0944"/>
+    <limit effort="100" velocity="6.54498" lower="-2.09440" upper="2.09440"/>
   </joint>
   <joint name="joint_6" type="revolute">
-    <!-- Flansch / Tool-Interface: ≈80 mm -->
-    <origin xyz="0 0 0.08" rpy="0 0 0"/>
     <parent link="Adept_Viper_s650_Link6"/>
     <child  link="Adept_Viper_650_Interface_Plate"/>
+    <origin xyz="0 0 0.08" rpy="0 0 0"/>
     <axis xyz="0 0 1"/>
-    <limit effort="100" velocity="10.47" lower="-3.1416" upper="3.1416"/>
+    <limit effort="100" velocity="10.47198" lower="-3.14159" upper="3.14159"/>
   </joint>
-  <!-- ===== Tool-Mount (kein TCP) ===== -->
+  <!-- TCP -->
   <link name="tool_mount"/>
   <joint name="tool_mount_joint" type="fixed">

Commit message: change robot colors

File: ws_moveit/src/omron_viper_description/urdf/omron_viper.urdf.xacro (robot description, xacro)
@@ -1,5 +1,8 @@
 <?xml version="1.0"?>
 <robot name="omron_viper_s650">
-  <!-- Welt -->
+  <!-- ===== Materialien ===== -->
+  <material name="Black"><color rgba="0 0 0 1"/></material>
+  <material name="White"><color rgba="1 1 1 1"/></material>
+  <!-- ===== Welt ===== -->
   <link name="world_mount"/>
   <joint name="world_to_base" type="fixed">
@@ -8,30 +11,40 @@
     <origin xyz="0 0 0" rpy="0 0 0"/>
   </joint>
-  <!-- Materialien -->
-  <material name="White"><color rgba="1 1 1 1"/></material>
-  <material name="Blue"><color rgba="0 0 1 1"/></material>
-  <material name="Red"><color rgba="1 0 0 1"/></material>
-  <material name="Green"><color rgba="0 1 0 1"/></material>
-  <material name="Gray"><color rgba="0.4 0.4 0.4 1"/></material>
-  <!-- LINKS (alle rpy=0) -->
+  <!-- ===== LINKS ===== -->
+  <!-- Link1 (Base) -> schwarz -->
   <link name="Adept_Viper_s650_Link1">
-    <visual><origin xyz="0 0 0" rpy="0 0 0"/><geometry>
-      <mesh filename="package://omron_viper_description/meshes/visual/Adept_Viper_650_Link1.stl"/>
-    </geometry><material name="White"/></visual>
-    <collision><origin xyz="0 0 0" rpy="0 0 0"/><geometry>
-      <mesh filename="package://omron_viper_description/meshes/collision/Adept_Viper_650_Link1.stl"/>
-    </geometry><material name="Blue"/></collision>
+    <visual>
+      <origin xyz="0 0 0" rpy="0 0 0"/>
+      <geometry>
+        <mesh filename="package://omron_viper_description/meshes/visual/Adept_Viper_650_Link1.stl"/>
+      </geometry>
+      <material name="Black"/>
+    </visual>
+    <collision>
+      <origin xyz="0 0 0" rpy="0 0 0"/>
+      <geometry>
+        <mesh filename="package://omron_viper_description/meshes/collision/Adept_Viper_650_Link1.stl"/>
+      </geometry>
+    </collision>
   </link>
+  <!-- Link2 -> weiß -->
   <link name="Adept_Viper_s650_Link2">
-    <visual><origin xyz="0 0 0" rpy="0 0 0"/><geometry>
-      <mesh filename="package://omron_viper_description/meshes/visual/Adept_Viper_650_Link2.stl"/>
-    </geometry><material name="Red"/></visual>
-    <collision><origin xyz="0 0 0" rpy="0 0 0"/><geometry>
-      <mesh filename="package://omron_viper_description/meshes/collision/Adept_Viper_650_Link2.stl"/>
-    </geometry><material name="Green"/></collision>
+    <visual>
+      <origin xyz="0 0 0" rpy="0 0 0"/>
+      <geometry>
+        <mesh filename="package://omron_viper_description/meshes/visual/Adept_Viper_650_Link2.stl"/>
+      </geometry>
+      <material name="White"/>
+    </visual>
+    <collision>
+      <origin xyz="0 0 0" rpy="0 0 0"/>
+      <geometry>
+        <mesh filename="package://omron_viper_description/meshes/collision/Adept_Viper_650_Link2.stl"/>
+      </geometry>
+    </collision>
   </link>
+  <!-- Link3 -> weiß (Mesh um Y 90°) -->
   <link name="Adept_Viper_s650_Link3">
     <visual>
-      <!-- Mesh 90° um Y drehen -->
       <origin xyz="0 0 0" rpy="0 1.5708 0"/>
       <geometry>
@@ -45,60 +58,71 @@
         <mesh filename="package://omron_viper_description/meshes/collision/Adept_Viper_650_Link3.stl"/>
       </geometry>
-      <material name="Blue"/>
     </collision>
   </link>
-<!-- Link4 -->
-<link name="Adept_Viper_s650_Link4">
-  <visual>
-    <origin xyz="0 0 0" rpy="0 -1.5708 0"/>
-    <geometry><mesh filename="package://omron_viper_description/meshes/visual/Adept_Viper_650_Link4.stl"/></geometry>
-    <material name="Red"/>
-  </visual>
-  <collision>
-    <origin xyz="0 0 0" rpy="0 -1.5708 0"/>
-    <geometry><mesh filename="package://omron_viper_description/meshes/collision/Adept_Viper_650_Link4.stl"/></geometry>
-    <material name="Blue"/>
-  </collision>
-</link>
-<!-- Link5 -->
-<link name="Adept_Viper_s650_Link5">
-  <visual>
-    <origin xyz="0 0 0" rpy="0 -1.5708 0"/>
-    <geometry><mesh filename="package://omron_viper_description/meshes/visual/Adept_Viper_650_Link5.stl"/></geometry>
-    <material name="Blue"/>
-  </visual>
-  <collision>
-    <origin xyz="0 0 0" rpy="0 -1.5708 0"/>
-    <geometry><mesh filename="package://omron_viper_description/meshes/collision/Adept_Viper_650_Link5.stl"/></geometry>
-    <material name="Blue"/>
-  </collision>
-</link>
-<!-- Link6 -->
-<link name="Adept_Viper_s650_Link6">
-  <visual>
-    <origin xyz="0 0 0" rpy="0 -1.5708 0"/>
-    <geometry><mesh filename="package://omron_viper_description/meshes/visual/Adept_Viper_650_Link6.stl"/></geometry>
-    <material name="Blue"/>
-  </visual>
-  <collision>
-    <origin xyz="0 0 0" rpy="0 -1.5708 0"/>
-    <geometry><mesh filename="package://omron_viper_description/meshes/collision/Adept_Viper_650_Link6.stl"/></geometry>
-    <material name="Blue"/>
-  </collision>
-</link>
-<!-- Interface Plate -->
-<link name="Adept_Viper_650_Interface_Plate">
-  <visual>
-    <origin xyz="0 0 0" rpy="0 -1.5708 0"/>
-    <geometry><mesh filename="package://omron_viper_description/meshes/visual/Adept_Viper_650_Interface_Plate.stl"/></geometry>
-    <material name="Gray"/>
-  </visual>
-  <collision>
-    <origin xyz="0 0 0" rpy="0 -1.5708 0"/>
-    <geometry><mesh filename="package://omron_viper_description/meshes/collision/Adept_Viper_650_Interface_Plate.stl"/></geometry>
-    <material name="Gray"/>
-  </collision>
-</link>
-  <!-- JOINTS (rein nach Datenblatt) -->
+  <!-- Link4 -> weiß (Mesh um Y -90°) -->
+  <link name="Adept_Viper_s650_Link4">
+    <visual>
+      <origin xyz="0 0 0" rpy="0 -1.5708 0"/>
+      <geometry>
+        <mesh filename="package://omron_viper_description/meshes/visual/Adept_Viper_650_Link4.stl"/>
+      </geometry>
+      <material name="White"/>
+    </visual>
+    <collision>
+      <origin xyz="0 0 0" rpy="0 -1.5708 0"/>
+      <geometry>
+        <mesh filename="package://omron_viper_description/meshes/collision/Adept_Viper_650_Link4.stl"/>
+      </geometry>
+    </collision>
+  </link>
+  <!-- Link5 -> weiß -->
+  <link name="Adept_Viper_s650_Link5">
+    <visual>
+      <origin xyz="0 0 0" rpy="0 -1.5708 0"/>
+      <geometry>
+        <mesh filename="package://omron_viper_description/meshes/visual/Adept_Viper_650_Link5.stl"/>
+      </geometry>
+      <material name="White"/>
+    </visual>
+    <collision>
+      <origin xyz="0 0 0" rpy="0 -1.5708 0"/>
+      <geometry>
+        <mesh filename="package://omron_viper_description/meshes/collision/Adept_Viper_650_Link5.stl"/>
+      </geometry>
+    </collision>
+  </link>
+  <!-- Link6 -> weiß -->
+  <link name="Adept_Viper_s650_Link6">
+    <visual>
+      <origin xyz="0 0 0" rpy="0 -1.5708 0"/>
+      <geometry>
+        <mesh filename="package://omron_viper_description/meshes/visual/Adept_Viper_650_Link6.stl"/>
+      </geometry>
+      <material name="White"/>
+    </visual>
+    <collision>
+      <origin xyz="0 0 0" rpy="0 -1.5708 0"/>
+      <geometry>
+        <mesh filename="package://omron_viper_description/meshes/collision/Adept_Viper_650_Link6.stl"/>
+      </geometry>
+    </collision>
+  </link>
+  <!-- Interface Plate -> weiß -->
+  <link name="Adept_Viper_650_Interface_Plate">
+    <visual>
+      <origin xyz="0 0 0" rpy="0 -1.5708 0"/>
+      <geometry>
+        <mesh filename="package://omron_viper_description/meshes/visual/Adept_Viper_650_Interface_Plate.stl"/>
+      </geometry>
+      <material name="White"/>
+    </visual>
+    <collision>
+      <origin xyz="0 0 0" rpy="0 -1.5708 0"/>
+      <geometry>
+        <mesh filename="package://omron_viper_description/meshes/collision/Adept_Viper_650_Interface_Plate.stl"/>
+      </geometry>
+    </collision>
+  </link>
+  <!-- ===== JOINTS (Datenblatt) ===== -->
   <joint name="joint_1" type="revolute">
     <parent link="Adept_Viper_s650_Link1"/>
@@ -143,5 +167,5 @@
     <limit effort="100" velocity="10.47198" lower="-3.14159" upper="3.14159"/>
   </joint>
-  <!-- TCP -->
+  <!-- ===== TCP ===== -->
   <link name="tool_mount"/>
   <joint name="tool_mount_joint" type="fixed">

Commit message: fix launch

File: ws_moveit/src/omron_viper_description/urdf/omron_viper.urdf.xacro (robot description, xacro)
@@ -5,7 +5,7 @@
   <material name="White"><color rgba="1 1 1 1"/></material>
   <!-- ===== Welt ===== -->
-  <link name="world_mount"/>
+  <link name="robot_mount"/>
   <joint name="world_to_base" type="fixed">
-    <parent link="world_mount"/>
+    <parent link="robot_mount"/>
     <child  link="Adept_Viper_s650_Link1"/>
     <origin xyz="0 0 0" rpy="0 0 0"/>

Commit message: save

File: ws_moveit/src/omron_viper_description/urdf/omron_viper.urdf.xacro (robot description, xacro)
@@ -168,9 +168,9 @@
   </joint>
   <!-- ===== TCP ===== -->
-  <link name="tool_mount"/>
-  <joint name="tool_mount_joint" type="fixed">
-    <parent link="Adept_Viper_650_Interface_Plate"/>
-    <child  link="tool_mount"/>
-    <origin xyz="0 0 0" rpy="0 0 0"/>
-  </joint>
+<link name="tool_mount"/>
+<joint name="tool_mount_joint" type="fixed">
+  <parent link="Adept_Viper_650_Interface_Plate"/>
+  <child  link="tool_mount"/>
+  <origin xyz="0 0 0" rpy="1.57079633 0 -1.57079633"/>
+</joint>
 </robot>

Commit message: save

File: ws_moveit/src/omron_viper_description/urdf/omron_viper.urdf.xacro (robot description, xacro)
@@ -217,5 +217,5 @@
     <parent link="sonotek_vortex"/>
     <child  link="tcp"/>
-    <origin xyz="0 0.05 -0.10" rpy="0 0 0"/>
+    <origin xyz="0 0.045 -0.11" rpy="0 0 0"/>
   </joint>
 </robot>
