Commit message: savew

File: ws_moveit/src/omron_moveit_config/config/omron_viper_s650.ros2_control.xacro (robot description, xacro)
@@ -1,54 +1,54 @@
 <?xml version="1.0"?>
 <robot xmlns:xacro="http://www.ros.org/wiki/xacro">
-    <xacro:macro name="omron_viper_s650_ros2_control" params="name initial_positions_file">
-        <xacro:property name="initial_positions" value="${xacro.load_yaml(initial_positions_file)['initial_positions']}"/>
-        <ros2_control name="${name}" type="system">
-            <hardware>
-                <!-- By default, set up controllers for simulation. This won't work on real hardware -->
-                <plugin>mock_components/GenericSystem</plugin>
-            </hardware>
-            <joint name="joint_1">
-                <command_interface name="position"/>
-                <state_interface name="position">
-                  <param name="initial_value">${initial_positions['joint_1']}</param>
-                </state_interface>
-                <state_interface name="velocity"/>
-            </joint>
-            <joint name="joint_2">
-                <command_interface name="position"/>
-                <state_interface name="position">
-                  <param name="initial_value">${initial_positions['joint_2']}</param>
-                </state_interface>
-                <state_interface name="velocity"/>
-            </joint>
-            <joint name="joint_3">
-                <command_interface name="position"/>
-                <state_interface name="position">
-                  <param name="initial_value">${initial_positions['joint_3']}</param>
-                </state_interface>
-                <state_interface name="velocity"/>
-            </joint>
-            <joint name="joint_4">
-                <command_interface name="position"/>
-                <state_interface name="position">
-                  <param name="initial_value">${initial_positions['joint_4']}</param>
-                </state_interface>
-                <state_interface name="velocity"/>
-            </joint>
-            <joint name="joint_5">
-                <command_interface name="position"/>
-                <state_interface name="position">
-                  <param name="initial_value">${initial_positions['joint_5']}</param>
-                </state_interface>
-                <state_interface name="velocity"/>
-            </joint>
-            <joint name="joint_6">
-                <command_interface name="position"/>
-                <state_interface name="position">
-                  <param name="initial_value">${initial_positions['joint_6']}</param>
-                </state_interface>
-                <state_interface name="velocity"/>
-            </joint>
-        </ros2_control>
-    </xacro:macro>
+  <!--
+    ros2_control-Konfiguration für Omron Viper S650
+    - Fake-Hardware mit mock_components/GenericSystem
+    - fake_sensor_commands=true => States folgen den Commands
+    - KEINE initial_positions mehr (erstmal alles 0.0)
+  -->
+  <xacro:macro name="omron_viper_s650_ros2_control" params="name">
+    <ros2_control name="${name}" type="system">
+      <hardware>
+        <plugin>mock_components/GenericSystem</plugin>
+        <!-- wichtig: Joint-States folgen den Kommandos -->
+        <param name="fake_sensor_commands">true</param>
+      </hardware>
+      <!-- Joint 1 -->
+      <joint name="joint_1">
+        <command_interface name="position"/>
+        <state_interface name="position"/>
+        <state_interface name="velocity"/>
+      </joint>
+      <!-- Joint 2 -->
+      <joint name="joint_2">
+        <command_interface name="position"/>
+        <state_interface name="position"/>
+        <state_interface name="velocity"/>
+      </joint>
+      <!-- Joint 3 -->
+      <joint name="joint_3">
+        <command_interface name="position"/>
+        <state_interface name="position"/>
+        <state_interface name="velocity"/>
+      </joint>
+      <!-- Joint 4 -->
+      <joint name="joint_4">
+        <command_interface name="position"/>
+        <state_interface name="position"/>
+        <state_interface name="velocity"/>
+      </joint>
+      <!-- Joint 5 -->
+      <joint name="joint_5">
+        <command_interface name="position"/>
+        <state_interface name="position"/>
+        <state_interface name="velocity"/>
+      </joint>
+      <!-- Joint 6 -->
+      <joint name="joint_6">
+        <command_interface name="position"/>
+        <state_interface name="position"/>
+        <state_interface name="velocity"/>
+      </joint>
+    </ros2_control>
+  </xacro:macro>
 </robot>

File: ws_moveit/src/omron_moveit_config/config/omron_viper_s650.urdf.xacro (robot description, xacro)
@@ -1,9 +1,9 @@
 <?xml version="1.0"?>
 <robot xmlns:xacro="http://www.ros.org/wiki/xacro" name="omron_viper_s650">
-    <xacro:arg name="initial_positions_file" default="initial_positions.yaml" />
-    <!-- Import omron_viper_s650 urdf file -->
-    <xacro:include filename="$(find omron_viper_description)/urdf/omron_viper.urdf.xacro" />
-    <!-- Import control_xacro -->
-    <xacro:include filename="omron_viper_s650.ros2_control.xacro" />
-    <xacro:omron_viper_s650_ros2_control name="FakeSystem" initial_positions_file="$(arg initial_positions_file)"/>
+  <!-- Basis-URDF aus dem Beschreibungspaket -->
+  <xacro:include filename="$(find omron_viper_description)/urdf/omron_viper.urdf.xacro" />
+  <!-- ros2_control-Xacro aus diesem Paket -->
+  <xacro:include filename="omron_viper_s650.ros2_control.xacro" />
+  <!-- FakeSystem für Simulation -->
+  <xacro:omron_viper_s650_ros2_control name="FakeSystem"/>
 </robot>

Commit message: save

File: ws_moveit/src/omron_moveit_config/config/omron_viper_s650.ros2_control.xacro (robot description, xacro)
@@ -4,12 +4,12 @@
     ros2_control-Konfiguration für Omron Viper S650
     - Fake-Hardware mit mock_components/GenericSystem
-    - fake_sensor_commands=true => States folgen den Commands
-    - KEINE initial_positions mehr (erstmal alles 0.0)
+    - fake_sensor_commands=true -> Joint-States folgen den Kommandos
+    - KEINE Macro-Parameter, alles fest verdrahtet
   -->
-  <xacro:macro name="omron_viper_s650_ros2_control" params="name">
-    <ros2_control name="${name}" type="system">
+  <xacro:macro name="omron_viper_s650_ros2_control">
+    <ros2_control name="omron_viper_s650_system" type="system">
       <hardware>
         <plugin>mock_components/GenericSystem</plugin>
-        <!-- wichtig: Joint-States folgen den Kommandos -->
+        <!-- States folgen direkt den Kommandos -->
         <param name="fake_sensor_commands">true</param>
       </hardware>
@@ -17,36 +17,36 @@
       <joint name="joint_1">
         <command_interface name="position"/>
-        <state_interface name="position"/>
-        <state_interface name="velocity"/>
+        <state_interface   name="position"/>
+        <state_interface   name="velocity"/>
       </joint>
       <!-- Joint 2 -->
       <joint name="joint_2">
         <command_interface name="position"/>
-        <state_interface name="position"/>
-        <state_interface name="velocity"/>
+        <state_interface   name="position"/>
+        <state_interface   name="velocity"/>
       </joint>
       <!-- Joint 3 -->
       <joint name="joint_3">
         <command_interface name="position"/>
-        <state_interface name="position"/>
-        <state_interface name="velocity"/>
+        <state_interface   name="position"/>
+        <state_interface   name="velocity"/>
       </joint>
       <!-- Joint 4 -->
       <joint name="joint_4">
         <command_interface name="position"/>
-        <state_interface name="position"/>
-        <state_interface name="velocity"/>
+        <state_interface   name="position"/>
+        <state_interface   name="velocity"/>
       </joint>
       <!-- Joint 5 -->
       <joint name="joint_5">
         <command_interface name="position"/>
-        <state_interface name="position"/>
-        <state_interface name="velocity"/>
+        <state_interface   name="position"/>
+        <state_interface   name="velocity"/>
       </joint>
       <!-- Joint 6 -->
       <joint name="joint_6">
         <command_interface name="position"/>
-        <state_interface name="position"/>
-        <state_interface name="velocity"/>
+        <state_interface   name="position"/>
+        <state_interface   name="velocity"/>
       </joint>
     </ros2_control>

File: ws_moveit/src/omron_moveit_config/config/omron_viper_s650.urdf.xacro (robot description, xacro)
@@ -5,5 +5,5 @@
   <!-- ros2_control-Xacro aus diesem Paket -->
   <xacro:include filename="omron_viper_s650.ros2_control.xacro" />
-  <!-- FakeSystem für Simulation -->
-  <xacro:omron_viper_s650_ros2_control name="FakeSystem"/>
+  <!-- ros2_control-System ohne Parameter -->
+  <xacro:omron_viper_s650_ros2_control/>
 </robot>

Commit message: save add nozzle

File: ws_moveit/src/omron_moveit_config/config/omron_viper_s650.ros2_control.xacro (robot description, xacro)
@@ -1,54 +1,54 @@
 <?xml version="1.0"?>
 <robot xmlns:xacro="http://www.ros.org/wiki/xacro">
-  <!--
-    ros2_control-Konfiguration für Omron Viper S650
-    - Fake-Hardware mit mock_components/GenericSystem
-    - fake_sensor_commands=true -> Joint-States folgen den Kommandos
-    - KEINE Macro-Parameter, alles fest verdrahtet
-  -->
-  <xacro:macro name="omron_viper_s650_ros2_control">
-    <ros2_control name="omron_viper_s650_system" type="system">
-      <hardware>
-        <plugin>mock_components/GenericSystem</plugin>
-        <!-- States folgen direkt den Kommandos -->
-        <param name="fake_sensor_commands">true</param>
-      </hardware>
-      <!-- Joint 1 -->
-      <joint name="joint_1">
-        <command_interface name="position"/>
-        <state_interface   name="position"/>
-        <state_interface   name="velocity"/>
-      </joint>
-      <!-- Joint 2 -->
-      <joint name="joint_2">
-        <command_interface name="position"/>
-        <state_interface   name="position"/>
-        <state_interface   name="velocity"/>
-      </joint>
-      <!-- Joint 3 -->
-      <joint name="joint_3">
-        <command_interface name="position"/>
-        <state_interface   name="position"/>
-        <state_interface   name="velocity"/>
-      </joint>
-      <!-- Joint 4 -->
-      <joint name="joint_4">
-        <command_interface name="position"/>
-        <state_interface   name="position"/>
-        <state_interface   name="velocity"/>
-      </joint>
-      <!-- Joint 5 -->
-      <joint name="joint_5">
-        <command_interface name="position"/>
-        <state_interface   name="position"/>
-        <state_interface   name="velocity"/>
-      </joint>
-      <!-- Joint 6 -->
-      <joint name="joint_6">
-        <command_interface name="position"/>
-        <state_interface   name="position"/>
-        <state_interface   name="velocity"/>
-      </joint>
-    </ros2_control>
-  </xacro:macro>
+    <xacro:macro name="omron_viper_s650_ros2_control" params="name initial_positions_file">
+        <xacro:property name="initial_positions" value="${xacro.load_yaml(initial_positions_file)['initial_positions']}"/>
+        <ros2_control name="${name}" type="system">
+            <hardware>
+                <!-- By default, set up controllers for simulation. This won't work on real hardware -->
+                <plugin>mock_components/GenericSystem</plugin>
+            </hardware>
+            <joint name="joint_1">
+                <command_interface name="position"/>
+                <state_interface name="position">
+                  <param name="initial_value">${initial_positions['joint_1']}</param>
+                </state_interface>
+                <state_interface name="velocity"/>
+            </joint>
+            <joint name="joint_2">
+                <command_interface name="position"/>
+                <state_interface name="position">
+                  <param name="initial_value">${initial_positions['joint_2']}</param>
+                </state_interface>
+                <state_interface name="velocity"/>
+            </joint>
+            <joint name="joint_3">
+                <command_interface name="position"/>
+                <state_interface name="position">
+                  <param name="initial_value">${initial_positions['joint_3']}</param>
+                </state_interface>
+                <state_interface name="velocity"/>
+            </joint>
+            <joint name="joint_4">
+                <command_interface name="position"/>
+                <state_interface name="position">
+                  <param name="initial_value">${initial_positions['joint_4']}</param>
+                </state_interface>
+                <state_interface name="velocity"/>
+            </joint>
+            <joint name="joint_5">
+                <command_interface name="position"/>
+                <state_interface name="position">
+                  <param name="initial_value">${initial_positions['joint_5']}</param>
+                </state_interface>
+                <state_interface name="velocity"/>
+            </joint>
+            <joint name="joint_6">
+                <command_interface name="position"/>
+                <state_interface name="position">
+                  <param name="initial_value">${initial_positions['joint_6']}</param>
+                </state_interface>
+                <state_interface name="velocity"/>
+            </joint>
+        </ros2_control>
+    </xacro:macro>
 </robot>

File: ws_moveit/src/omron_moveit_config/config/omron_viper_s650.urdf.xacro (robot description, xacro)
@@ -1,9 +1,9 @@
 <?xml version="1.0"?>
 <robot xmlns:xacro="http://www.ros.org/wiki/xacro" name="omron_viper_s650">
-  <!-- Basis-URDF aus dem Beschreibungspaket -->
-  <xacro:include filename="$(find omron_viper_description)/urdf/omron_viper.urdf.xacro" />
-  <!-- ros2_control-Xacro aus diesem Paket -->
-  <xacro:include filename="omron_viper_s650.ros2_control.xacro" />
-  <!-- ros2_control-System ohne Parameter -->
-  <xacro:omron_viper_s650_ros2_control/>
+    <xacro:arg name="initial_positions_file" default="initial_positions.yaml" />
+    <!-- Import omron_viper_s650 urdf file -->
+    <xacro:include filename="$(find omron_viper_description)/urdf/omron_viper.urdf.xacro" />
+    <!-- Import control_xacro -->
+    <xacro:include filename="omron_viper_s650.ros2_control.xacro" />
+    <xacro:omron_viper_s650_ros2_control name="FakeSystem" initial_positions_file="$(arg initial_positions_file)"/>
 </robot>

File: ws_moveit/src/omron_viper_description/urdf/omron_viper.urdf.xacro (robot description, xacro)
@@ -179,10 +179,43 @@
     <limit effort="100" velocity="10.47198" lower="-3.14159" upper="3.14159"/>
   </joint>
-  <!-- TCP-Fixgelenk -->
+  <!-- tool_mount: neutrale Orientierung auf der Interface-Plate -->
   <joint name="tool_mount_joint" type="fixed">
     <parent link="Adept_Viper_650_Interface_Plate"/>
     <child  link="tool_mount"/>
-    <!-- TCP-Ausrichtung wie von dir gewünscht -->
+    <origin xyz="0 0 0" rpy="0 0 0"/>
+  </joint>
+  <!-- Sonotek Vortex Nozzle (Mesh in mm -> scale auf Meter) -->
+  <link name="sonotek_vortex">
+    <visual>
+      <!-- Nur das Mesh ist rotiert, KEINE Verschiebung -->
+      <origin xyz="0 0 0" rpy="0 1.57079633 0"/>
+      <geometry>
+        <mesh filename="package://omron_viper_description/meshes/tools/Sonotek_Vortex.stl"
+              scale="0.001 0.001 0.001"/>
+      </geometry>
+      <material name="White"/>
+    </visual>
+    <collision>
+      <origin xyz="0 0 0" rpy="0 1.57079633 0"/>
+      <geometry>
+        <mesh filename="package://omron_viper_description/meshes/tools/Sonotek_Vortex.stl"
+              scale="0.001 0.001 0.001"/>
+      </geometry>
+    </collision>
+  </link>
+  <!-- Joint: tool_mount -> mesh (nur Rotation im TF, keine Verschiebung) -->
+  <joint name="sonotek_vortex_joint" type="fixed">
+    <parent link="tool_mount"/>
+    <child  link="sonotek_vortex"/>
+    <!-- TF-Ausrichtung zwischen Flansch und Tool -->
     <origin xyz="0 0 0" rpy="1.57079633 0 -1.57079633"/>
   </joint>
+  <!-- TCP-Link: nur Frame, kein Mesh -->
+  <link name="tcp"/>
+  <!-- Joint: sonotek_vortex -> tcp (hier: -10cm in z, +5cm in y) -->
+  <joint name="tcp_joint" type="fixed">
+    <parent link="sonotek_vortex"/>
+    <child  link="tcp"/>
+    <origin xyz="0 0.05 -0.10" rpy="0 0 0"/>
+  </joint>
 </robot>
