Commit message: save

File: ws_moveit/src/omron_moveit_config/config/omron_viper_s650.ros2_control.xacro (robot description, xacro)
@@ -1,54 +1,91 @@
 <?xml version="1.0"?>
 <robot xmlns:xacro="http://www.ros.org/wiki/xacro">
-    <xacro:macro name="omron_viper_s650_ros2_control" params="name initial_positions_file">
-        <xacro:property name="initial_positions" value="${xacro.load_yaml(initial_positions_file)['initial_positions']}"/>
-        <ros2_control name="${name}" type="system">
-            <hardware>
-                <!-- By default, set up controllers for simulation. This won't work on real hardware -->
-                <plugin>mock_components/GenericSystem</plugin>
-            </hardware>
-            <joint name="joint_1">
-                <command_interface name="position"/>
-                <state_interface name="position">
-                  <param name="initial_value">${initial_positions['joint_1']}</param>
-                </state_interface>
-                <state_interface name="velocity"/>
-            </joint>
-            <joint name="joint_2">
-                <command_interface name="position"/>
-                <state_interface name="position">
-                  <param name="initial_value">${initial_positions['joint_2']}</param>
-                </state_interface>
-                <state_interface name="velocity"/>
-            </joint>
-            <joint name="joint_3">
-                <command_interface name="position"/>
-                <state_interface name="position">
-                  <param name="initial_value">${initial_positions['joint_3']}</param>
-                </state_interface>
-                <state_interface name="velocity"/>
-            </joint>
-            <joint name="joint_4">
-                <command_interface name="position"/>
-                <state_interface name="position">
-                  <param name="initial_value">${initial_positions['joint_4']}</param>
-                </state_interface>
-                <state_interface name="velocity"/>
-            </joint>
-            <joint name="joint_5">
-                <command_interface name="position"/>
-                <state_interface name="position">
-                  <param name="initial_value">${initial_positions['joint_5']}</param>
-                </state_interface>
-                <state_interface name="velocity"/>
-            </joint>
-            <joint name="joint_6">
-                <command_interface name="position"/>
-                <state_interface name="position">
-                  <param name="initial_value">${initial_positions['joint_6']}</param>
-                </state_interface>
-                <state_interface name="velocity"/>
-            </joint>
-        </ros2_control>
-    </xacro:macro>
+  <!--
+    Macro für ros2_control:
+      - name: Name des ros2_control-Systems (z.B. "omron_viper_s650_system")
+      - initial_positions_file: YAML-Datei mit Abschnitt "initial_positions"
+           initial_positions:
+             joint_1: 0.0
+             joint_2: 0.0
+             ...
+  -->
+  <xacro:macro name="omron_viper_s650_ros2_control" params="name initial_positions_file">
+    <!-- YAML mit Startpositionen laden -->
+    <xacro:property
+        name="initial_positions"
+        value="${xacro.load_yaml(initial_positions_file)['initial_positions']}" />
+    <ros2_control name="${name}" type="system">
+      <hardware>
+        <!-- Fake-System für Simulation -->
+        <plugin>mock_components/GenericSystem</plugin>
+        <param name="fake_sensor_commands">true</param>
+      </hardware>
+      <!-- Joint 1 -->
+      <joint name="joint_1">
+        <command_interface name="position">
+          <param name="min">-6.283185307</param>
+          <param name="max"> 6.283185307</param>
+        </command_interface>
+        <state_interface name="position">
+          <param name="initial_value">${initial_positions['joint_1']}</param>
+        </state_interface>
+        <state_interface name="velocity"/>
+      </joint>
+      <!-- Joint 2 -->
+      <joint name="joint_2">
+        <command_interface name="position">
+          <param name="min">-6.283185307</param>
+          <param name="max"> 6.283185307</param>
+        </command_interface>
+        <state_interface name="position">
+          <param name="initial_value">${initial_positions['joint_2']}</param>
+        </state_interface>
+        <state_interface name="velocity"/>
+      </joint>
+      <!-- Joint 3 -->
+      <joint name="joint_3">
+        <command_interface name="position">
+          <param name="min">-6.283185307</param>
+          <param name="max"> 6.283185307</param>
+        </command_interface>
+        <state_interface name="position">
+          <param name="initial_value">${initial_positions['joint_3']}</param>
+        </state_interface>
+        <state_interface name="velocity"/>
+      </joint>
+      <!-- Joint 4 -->
+      <joint name="joint_4">
+        <command_interface name="position">
+          <param name="min">-6.283185307</param>
+          <param name="max"> 6.283185307</param>
+        </command_interface>
+        <state_interface name="position">
+          <param name="initial_value">${initial_positions['joint_4']}</param>
+        </state_interface>
+        <state_interface name="velocity"/>
+      </joint>
+      <!-- Joint 5 -->
+      <joint name="joint_5">
+        <command_interface name="position">
+          <param name="min">-6.283185307</param>
+          <param name="max"> 6.283185307</param>
+        </command_interface>
+        <state_interface name="position">
+          <param name="initial_value">${initial_positions['joint_5']}</param>
+        </state_interface>
+        <state_interface name="velocity"/>
+      </joint>
+      <!-- Joint 6 -->
+      <joint name="joint_6">
+        <command_interface name="position">
+          <param name="min">-6.283185307</param>
+          <param name="max"> 6.283185307</param>
+        </command_interface>
+        <state_interface name="position">
+          <param name="initial_value">${initial_positions['joint_6']}</param>
+        </state_interface>
+        <state_interface name="velocity"/>
+      </joint>
+    </ros2_control>
+  </xacro:macro>
 </robot>

File: ws_moveit/src/omron_moveit_config/config/omron_viper_s650.urdf.xacro (robot description, xacro)
@@ -1,9 +1,22 @@
 <?xml version="1.0"?>
 <robot xmlns:xacro="http://www.ros.org/wiki/xacro" name="omron_viper_s650">
-    <xacro:arg name="initial_positions_file" default="initial_positions.yaml" />
-    <!-- Import omron_viper_s650 urdf file -->
-    <xacro:include filename="$(find omron_viper_description)/urdf/omron_viper.urdf.xacro" />
-    <!-- Import control_xacro -->
-    <xacro:include filename="omron_viper_s650.ros2_control.xacro" />
-    <xacro:omron_viper_s650_ros2_control name="FakeSystem" initial_positions_file="$(arg initial_positions_file)"/>
+  <!--
+    Pfad zur Datei mit den Initialpositionen.
+    Bitte ggf. den Paketnamen/Pfad anpassen, falls deine initial_positions.yaml woanders liegt.
+  -->
+  <xacro:arg
+      name="initial_positions_file"
+      default="$(find omron_moveit_config)/config/initial_positions.yaml" />
+  <!-- Basis-URDF aus dem Beschreibungspaket -->
+  <xacro:include filename="$(find omron_viper_description)/urdf/omron_viper.urdf.xacro" />
+  <!-- ros2_control-Xacro aus diesem Paket -->
+  <xacro:include filename="omron_viper_s650.ros2_control.xacro" />
+  <!--
+    ros2_control-System:
+      - Name: omron_viper_s650_system
+      - Initialpositionen aus initial_positions_file
+  -->
+  <xacro:omron_viper_s650_ros2_control
+      name="omron_viper_s650_system"
+      initial_positions_file="$(arg initial_positions_file)" />
 </robot>

Commit message: save

File: ws_moveit/src/omron_moveit_config/config/omron_viper_s650.ros2_control.xacro (robot description, xacro)
@@ -4,12 +4,12 @@
     Macro für ros2_control:
       - name: Name des ros2_control-Systems (z.B. "omron_viper_s650_system")
-      - initial_positions_file: YAML-Datei mit Abschnitt "initial_positions"
-           initial_positions:
-             joint_1: 0.0
-             joint_2: 0.0
-             ...
+      - initial_positions werden intern aus
+        $(find omron_moveit_config)/config/initial_positions.yaml geladen.
   -->
-  <xacro:macro name="omron_viper_s650_ros2_control" params="name initial_positions_file">
+  <xacro:macro name="omron_viper_s650_ros2_control" params="name">
     <!-- YAML mit Startpositionen laden -->
+    <xacro:property
+        name="initial_positions_file"
+        value="$(find omron_moveit_config)/config/initial_positions.yaml" />
     <xacro:property
         name="initial_positions"

File: ws_moveit/src/omron_moveit_config/config/omron_viper_s650.urdf.xacro (robot description, xacro)
@@ -1,22 +1,12 @@
 <?xml version="1.0"?>
 <robot xmlns:xacro="http://www.ros.org/wiki/xacro" name="omron_viper_s650">
-  <!--
-    Pfad zur Datei mit den Initialpositionen.
-    Bitte ggf. den Paketnamen/Pfad anpassen, falls deine initial_positions.yaml woanders liegt.
-  -->
-  <xacro:arg
-      name="initial_positions_file"
-      default="$(find omron_moveit_config)/config/initial_positions.yaml" />
   <!-- Basis-URDF aus dem Beschreibungspaket -->
   <xacro:include filename="$(find omron_viper_description)/urdf/omron_viper.urdf.xacro" />
   <!-- ros2_control-Xacro aus diesem Paket -->
   <xacro:include filename="omron_viper_s650.ros2_control.xacro" />
-  <!--
-    ros2_control-System:
-      - Name: omron_viper_s650_system
-      - Initialpositionen aus initial_positions_file
-  -->
+  <!-- ros2_control-System:
+       - Name: omron_viper_s650_system
+       - Initialpositionen werden *intern* geladen -->
   <xacro:omron_viper_s650_ros2_control
-      name="omron_viper_s650_system"
-      initial_positions_file="$(arg initial_positions_file)" />
+      name="omron_viper_s650_system" />
 </robot>
